File: RJ10Adapter.kicad_sch (KiCad schematic)
At the start: 11 parts, among them J1 RJ10, J2 Conn_01x06_Male, J3 USB_B_Micro, SW1 SW_Push, U1 AMS1117-3.3, U2 ESP-12F

Commit message: v1.4
Parts:
- C1, C2: footprint Capacitor_SMD:C_0805_2012Metric_Pad1.15x1.40mm_HandSolder -> Capacitor_SMD:C_0805_2012Metric_Pad1.18x1.45mm_HandSolder
- R1, R2, R3: footprint Resistor_SMD:R_0805_2012Metric_Pad1.15x1.40mm_HandSolder -> Resistor_SMD:R_0805_2012Metric_Pad1.20x1.40mm_HandSolder
